File: tedy_PCB/tedy.brd (EAGLE design)
At the start: 65 x 75 mm, 27 parts, among them IC1 TP4056, T1 DMN3024LSD

Commit message: update on 16-2-2019
Parts:
- removed BAT, POW_S: (no value), custom_package:CONNECTOR_1.5MM_THROUGH_HOLE_(2_PIN)
- removed IC1: TP4056, TP4056:SOP-8
- removed LED_C, LED_P: (no value), led:CHIP-LED0805
- added B+: B+, custom_package:PIN_1
- added B-: B-, custom_package:PIN_1
- added C2: 0.1u, resistor:C0805
- added C5: 22u, resistor:C0805
- added D1, D2, D3: SS24, custom_package:SS24
- added L1: 22uH, custom_package:4D28
- added LED_: (no value), custom_package:2_COLOUR_LED
- added MT3608: MT3608, custom_package:SOT23-6
- added POWER_SWITCH: 6PIN_SWITCH, custom_package:6PIN_SWITCH
- added Q1: DMP1045U, custom_package:SOT23-3
- added R1, R8: 1k, resistor:R0805
- added R9: 7.5k, resistor:R0805
- added TP4056: TP4056, TP4056:SOP-8
- C1: value 0.1u -> 0.1uF; device eagle-ltspice:C0805 -> resistor:C0805
- C3: device eagle-ltspice:C0805 -> resistor:C0805
- C4: value 0.1u -> 22uF; device eagle-ltspice:C0805 -> resistor:C0805
- DW01: value (none) -> DW01
- R3: value 1k -> 1.2k
- R4: value 1.2k -> 1k; device adafruit:R0805 -> resistor:R0805
- R6: value 1k -> 100k; device adafruit:R0805 -> resistor:R0805
- moved DW01 115.9 mm to (0.00, -52.0), flipped to the top, turned to 0 degrees
- moved C3 97.1 mm to (14.0, -45.0), flipped to the top, turned to 0 degrees
- moved R4 96.9 mm to (31.0, -45.0), flipped to the top, turned to 0 degrees
- moved R5 96.2 mm to (4.00, -45.0), flipped to the top
- moved C4 94.6 mm to (-1.00, -45.0), flipped to the top, turned to 0 degrees
- moved R6 88.8 mm to (19.0, -37.0), flipped to the top
- moved C1 83.9 mm to (25.0, -37.0), flipped to the top, turned to 0 degrees
- moved R2 75.6 mm to (27.0, -45.0)
- moved T1 66.0 mm to (34.0, -9.00), flipped to the top, turned to 0 degrees
- moved R3 64.0 mm to (31.0, -37.0)
Connections:
- removed net B+: BAT.1, C4.1, IC1.5, POW_S.1, R5.2
- removed net B-: BAT.2, T1.2, T1.3
- removed net N$10 (its old number): IC1.7, R2.1
- removed net N$20: DW01.2, R6.1
- removed net N$9 (its old number): IC1.6, R3.1
- new net N$14: C3.1, R5.2
- new net N$17: D1.2, POWER_SWITCH.2
- new net N$18: C5.1, D2.2, D3.1, R9.2
- new net N$19: D2.1, L1.P$2, MT3608.1
- new net N$2: LED_.1, R1.1
- new net N$3: LED_.3, R2.1
- new net N$4: R3.2, TP4056.2
- new net N$5: R1.2, TP4056.6
- new net N$6: DW01.2, R4.2
- new net N$7: R2.2, TP4056.7
- new net V3.7: C4.1, L1.P$1, MT3608.4, MT3608.5, POWER_SWITCH.5, POWER_SWITCH.6, Q1.2
- new net V5: C1.1, D1.1, LED_.2, LED_.4, Q1.1, R6.2, TP4056.4, TP4056.8, USB3.1_TYPE-C.A4, USB3.1_TYPE-C.A9, USB3.1_TYPE-C.B4, USB3.1_TYPE-C.B9
- net DM: no longer USB3.1_TYPE-C.A7, USB3.1_TYPE-C.B7
- net DP: no longer USB3.1_TYPE-C.A6, USB3.1_TYPE-C.B6
- net GND: now also C3.2, C5.2, MT3608.2, R3.1, R4.1, R6.1, R8.1, TP4056.1, TP4056.3; no longer IC1.1, IC1.3, R4.2, R6.2
- net N$11: now also C2.2, DW01.6; no longer LED_P.C, R3.2
- net N$12: now also C2.1, DW01.5, R5.1; no longer LED_C.C, R2.2
- net N$13: now also B+.1, Q1.3, TP4056.5; no longer IC1.2, R4.1
- net N$15: now also B-.1, T1.2, T1.3; no longer C3.1, DW01.6
- net N$16: now also MT3608.3, R8.2, R9.1; no longer C3.2, DW01.5, R5.1
- net VCC: now also D3.2, POWER_SWITCH.3; no longer POW_S.2
- net VIN: no longer C1.1, IC1.4, IC1.8, LED_C.A, LED_P.A, USB3.1_TYPE-C.A4, USB3.1_TYPE-C.A9, USB3.1_TYPE-C.B4, USB3.1_TYPE-C.B9
Routing:
- net VCC: track 190.6 -> 0.00 mm
- net VIN: track 156.2 -> 0.00 mm, vias 3 -> 0
- net B+: track 122.1 -> 0.00 mm, vias 1 -> 0
- net RXD: track 97.8 -> 0.00 mm
- net TXD: track 90.7 -> 0.00 mm
- net B-: track 82.1 -> 0.00 mm, vias 1 -> 0
- net DP: track 76.4 -> 0.00 mm, vias 1 -> 0
- net DM: track 75.9 -> 0.00 mm, vias 2 -> 0
- net N$29: track 66.7 -> 0.00 mm, vias 1 -> 0
- net N$25: track 65.0 -> 0.00 mm
- net N$9 (its old number): track 54.8 -> 0.00 mm, vias 1 -> 0
- net N$10 (its old number): track 52.5 -> 0.00 mm, vias 1 -> 0
- net N$24: track 50.5 -> 0.00 mm
- net GND: track 36.7 -> 0.00 mm, vias 6 -> 0
- net SCL: track 32.4 -> 0.00 mm
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