File: tedy_PCB/tedy.sch (EAGLE design)
At the start: 27 parts, among them IC1 TP4056, T1 DMN3024LSD

Commit message: update on 16-2-2019
Parts:
- removed BAT, POW_S: (no value), custom_package:CONNECTOR_1.5MM_THROUGH_HOLE_(2_PIN)
- removed IC1: TP4056, TP4056:TP4056
- removed LED_C, LED_P: (no value), led:LEDCHIP-LED0805
- added B+: B+, custom_package:PIN_1
- added B-: B-, custom_package:PIN_1
- added C2: 0.1u, resistor:C-USC0805
- added C5: 22u, resistor:C-USC0805
- added D1, D2, D3: SS24, custom_package:SS24
- added L1: 22uH, custom_package:4D28
- added LED_: (no value), custom_package:2_COLOUR_LED
- added MT3608: MT3608, custom_package:MT3608
- added POWER_SWITCH: 6PIN_SWITCH, custom_package:6PIN_SWITCH
- added Q1: DMP1045U, custom_package:DMP1045U
- added R1, R8: 1k, resistor:R-US_R0805
- added R9: 7.5k, resistor:R-US_R0805
- added TP4056: TP4056, TP4056:TP4056
- C1: value 0.1u -> 0.1uF; device eagle-ltspice:C -> resistor:C-USC0805
- C3: device eagle-ltspice:C -> resistor:C-USC0805
- C4: value 0.1u -> 22uF; device eagle-ltspice:C -> resistor:C-USC0805
- R3: value 1k -> 1.2k
- R4: value 1.2k -> 1k; device adafruit:R-US_R0805 -> resistor:R-US_R0805
- R6: value 1k -> 100k; device adafruit:R-US_R0805 -> resistor:R-US_R0805
Connections:
- removed net B+: BAT.1, C4.1, IC1.BAT, POW_S.1, R5.2
- removed net B-: BAT.2, T1A.S
- removed net N$10 (its old number): IC1.CHRG, R2.1
- removed net N$20: DW01.CS, R6.1
- removed net N$9 (its old number): IC1.STDBY, R3.1
- new net N$14: C3.1, R5.2
- new net N$17: D1.C, POWER_SWITCH.P
- new net N$18: C5.1, D2.C, D3.A, R9.2
- new net N$19: D2.A, L1.2, MT3608.SW
- new net N$2: LED_R.1, R1.1
- new net N$3: LED_G.1, R2.1
- new net N$4: R3.2, TP4056.PROG
- new net N$5: R1.2, TP4056.STDBY
- new net N$6: DW01.CS, R4.2
- new net N$7: R2.2, TP4056.CHRG
- new net V3.7: C4.1, L1.1, MT3608.EN, MT3608.IN, POWER_SWITCH.P1, POWER_SWITCH.S1, Q1.S
- new net V5: C1.1, D1.A, LED_G.2, LED_R.2, Q1.G, R6.2, TP4056.CE, TP4056.VCC, USB3.1_TYPE-C.A4, USB3.1_TYPE-C.A9, USB3.1_TYPE-C.B4, USB3.1_TYPE-C.B9
- net DM: no longer USB3.1_TYPE-C.A7, USB3.1_TYPE-C.B7
- net DP: no longer USB3.1_TYPE-C.A6, USB3.1_TYPE-C.B6
- net GND: now also C3.2, C5.2, MT3608.GND, R3.1, R4.1, R6.1, R8.1, TP4056.GND, TP4056.TEMP; no longer IC1.GND, IC1.TEMP, R4.2, R6.2
- net N$11: now also C2.2, DW01.GND; no longer LED_P.C, R3.2
- net N$12: now also C2.1, DW01.VCC, R5.1; no longer LED_C.C, R2.2
- net N$13: now also B+.1, Q1.D, TP4056.BAT; no longer IC1.PROG, R4.1
- net N$15: now also B-.1, T1A.S; no longer C3.1, DW01.GND
- net N$16: now also MT3608.FB, R8.2, R9.1; no longer C3.2, DW01.VCC, R5.1
- net VCC: now also D3.C, POWER_SWITCH.S; no longer POW_S.2
- net VIN: no longer C1.1, IC1.CE, IC1.VCC, LED_C.A, LED_P.A, USB3.1_TYPE-C.A4, USB3.1_TYPE-C.A9, USB3.1_TYPE-C.B4, USB3.1_TYPE-C.B9
Other:
- note removed: "B+"
- note removed: "B-"
- moved on the sheet: C1, C3, C4, MIC, NFC_PORT, R2, R3, R4, R5, R6, SPEAKER, T1A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
